File: hardware/logicboard/bui-001.sch (EAGLE design)
At the start: 28 parts, among them IC1 5V, IC2 74LS07N, IC3 4066N, K1 G5V1, T1 2SC1815, U1 DS18B20

Commit message: Initial version of schematic.
Parts:
- removed C4, C5, C6: 103, rcl:C-US025-025X050
- removed D1, D2: DIODE-1N4148, SparkFun-DiscreteSemi:DIODE-1N4148
- removed IC3: 4066N, 40xx:4066N
- removed JP2: (no value), pinhead:PINHD-1X2
- removed K1: G5V1, relay:G5V1
- removed OK1: 6N137, optocoupler:6N137
- removed RN2: 330, resistor-net:RN08
- removed RN3: 4.7k, resistor-net:RN08
- removed RN4: 10k, resistor-net:RN04
- removed SV2: (no value), con-ml:ML20LE
- removed T1: 2SC1815, transistor:2SC1815
- removed U1: DS18B20, SparkFun-Sensors:DS18B20
- added J1: DIN5, SparkFun-Connectors:DIN5
- R1: value 1k -> 220
- R2: value 47k -> 220
- RN1: value 220 -> 10k; device resistor-dil:8R-N -> resistor-net:RN08
- SV1: device con-ml:ML34LE -> con-ml:ML14LE
Connections:
- removed net A1: IC3A.B, MC1.A0, SV1-4.S
- removed net A2: IC3B.B, MC1.A1, SV1-10.S
- removed net A3: IC3C.B, MC1.A2, SV1-16.S
- removed net A4: IC3D.B, MC1.A3, SV1-22.S
- removed net D1: MC1.6, RN3.4, SV1-3.S
- removed net D2: MC1.9, RN3.5, SV1-9.S
- removed net D3: MC1.10, RN3.6, SV1-15.S
- removed net D4: MC1.12, RN3.7, SV1-21.S
- removed net LED0: IC2D.I, MC1.13, SV1-25.S
- removed net LED0K: RN2.2, SV1-26.S
- removed net LED1: MC1.4, SV1-27.S
- removed net LED1K: RN2.3, SV1-28.S
- removed net LED2: IC2E.I, MC1.5, SV1-29.S
- removed net LED2K: RN2.4, SV1-30.S
- removed net LED3: MC1.8, SV1-31.S
- removed net LED3K: RN2.5, SV1-32.S
- removed net LED4: IC2F.I, MC1.11, SV1-33.S
- removed net LED4K: RN2.6, SV1-34.S
- removed net MIDIINSND: D1.C, OK1.A, RN1A.1
- removed net MIDIOUT2RTN: IC2C.O, RN1G.1
- removed net MIDIOUTRTN: IC2B.O, RN1E.1
- removed net MIDITHRURTN: IC2A.O, RN1C.1
- removed net MINRTN: D1.A, OK1.C, SV2-6.S
- removed net MINSND: RN1A.2, SV2-5.S
- removed net MO1RTN: RN1E.2, SV2-11.S
- removed net MO1SND: RN1D.2, SV2-10.S
- removed net MO2RTN: RN1G.2, SV2-16.S
- removed net MO2SND: RN1F.2, SV2-15.S
- removed net MTHRTN: RN1C.2, SV2-18.S
- removed net MTHSND: RN1B.2, SV2-17.S
- removed net PULLUP: IC3A.C, IC3B.C, IC3C.C, IC3D.C, MC1.7
- removed net RLY: MC1.A5, R1.2
- removed net RLYDRV: R1.1, R2.2, T1.B
- removed net RLYSNK: D2.A, K11.2, T1.C
- removed net RST: MC1.R@1, SV2-3.S
- removed net RX: IC2A.I, MC1.RX, OK1.VO
- removed net SCL: MC1.3, RN3.3, SV1-12.S, SV1-18.S, SV1-24.S, SV1-6.S
- removed net SDA: MC1.2, RN3.2, SV1-11.S, SV1-17.S, SV1-23.S, SV1-5.S
- removed net THS: MC1.A4, RN3.8, SV2-9.S, U1.DQ
- removed net TX: IC2B.I, IC2C.I, MC1.TX
- removed net VDD: MC1.3V, SV2-19.S
- removed net XLEDB: IC2E.O, SV2-13.S
- removed net XLEDG: IC2D.O, SV2-12.S
- removed net XLEDR: IC2F.O, SV2-14.S
- new net N$1: MC1.A5, RN1.7, SV1-11.S
- new net N$10: J1.4, R1.2
- new net N$2: MC1.A4, RN1.6, SV1-9.S
- new net N$7: IC2A.I, MC1.TX
- new net N$8: IC2A.O, R2.1
- new net N$9: J1.5, R2.2
- net +12V: no longer JP2.1, K12.O, SV2-1.S
- net 12VRLY: no longer JP2.2, K12.P, K12.P@1
- net GND: now also IC2B.I, IC2C.I, IC2D.I, IC2E.I, IC2F.I, J1.2, SV1-10.S, SV1-12.S, SV1-4.S, SV1-6.S; no longer C4.2, C5.2, C6.2, IC3P.VSS, R2.1, RN2.1, SV1-20.S, SV2-2.S, SV2-20.S, SV2-4.S, SV2-8.S, T1.E, U1.GND
- net N$3: now also MC1.A3, RN1.5, SV1-7.S; no longer IC3A.A, RN4.2
- net N$4: now also MC1.A2, RN1.4, SV1-5.S; no longer IC3B.A, RN4.3
- net N$5: now also MC1.A1, RN1.3, SV1-3.S; no longer IC3C.A, RN4.4
- net N$6: now also MC1.A0, RN1.2, SV1-1.S; no longer IC3D.A, RN4.5
- net VCC: now also R1.1; no longer C4.1, C5.1, C6.1, D2.C, IC3P.VDD, K11.1, OK1.VE, RN1B.1, RN1D.1, RN1F.1, RN3.1, RN4.1, SV2-7.S, U1.VDD
- net VOUT: now also RN1.1; no longer SV1-1.S, SV1-13.S, SV1-19.S, SV1-7.S
Other:
- note removed: "Pineapple II 2.0.2"
- moved on the sheet: C1, C2, C3, IC1, IC2A, IC2B, IC2C, IC2D, IC2E, IC2F, JP1, R1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

Commit message: Finished schematic.
Connections:
- removed net 12VRLY: C1.1, IC1.IN
- removed net N$1: MC1.A5, RN1.7, SV1-11.S
- removed net N$2: MC1.A4, RN1.6, SV1-9.S
- removed net N$3: MC1.A3, RN1.5, SV1-7.S
- removed net N$4: MC1.A2, RN1.4, SV1-5.S
- removed net N$5: MC1.A1, RN1.3, SV1-3.S
- removed net N$6: MC1.A0, RN1.2, SV1-1.S
- new net ANALOG0: MC1.A0, RN1.2, SV1-3.S
- new net ANALOG1: MC1.A1, RN1.3, SV1-5.S
- new net ANALOG2: MC1.A2, RN1.4, SV1-7.S
- new net ANALOG3: MC1.A3, RN1.5, SV1-9.S
- new net ANALOG4: MC1.A4, RN1.6, SV1-11.S
- new net ANALOG5: MC1.A5, RN1.7, SV1-13.S
- net +12V: now also C1.1, IC1.IN
Other:
- moved on the sheet: SV1-1, SV1-11, SV1-13, SV1-3, SV1-5, SV1-7, SV1-9

Commit message: INT switch.
Parts:
- added S1: MOMENTARY-SWITCH-SPST-PTH-6.0MM, SparkFun-Switches:MOMENTARY-SWITCH-SPST-PTH-6.0MM
Connections:
- new net N$1: MC1.2, S1.2
- net GND: now also S1.1
Changed lines of the file:
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@@
 <part name="SUPPLY23" library="supply2" deviceset="GND" device=""/>
 <part name="RN1" library="resistor-net" library_urn="urn:adsk.eagle:library:343" deviceset="RN08" device="" package3d_urn="urn:adsk.eagle:package:24977/1" value="10k"/>
-<part name="R1" library="resistor" library_urn="urn:adsk.eagle:library:348" deviceset="R-EU_" device="0204/5" package3d_urn="urn:adsk.eagle:package:25955/1" value="220"/>
-<part name="R2" library="resistor" library_urn="urn:adsk.eagle:library:348" deviceset="R-EU_" device="0204/5" package3d_urn="urn:adsk.eagle:package:25955/1" value="220"/>
+<part name="R1" library="resistor" library_urn="urn:adsk.eagle:library:348" deviceset="R-EU_" device="0204/5" package3d_urn="urn:adsk.eagle:package:23488/1" value="220"/>
+<part name="R2" library="resistor" library_urn="urn:adsk.eagle:library:348" deviceset="R-EU_" device="0204/5" package3d_urn="urn:adsk.eagle:package:23488/1" value="220"/>
 <part name="J1" library="SparkFun-Connectors" library_urn="urn:adsk.eagle:library:513" deviceset="DIN5" device="" package3d_urn="urn:adsk.eagle:package:38294/1"/>
 <part name="SUPPLY1" library="supply2" deviceset="GND" device=""/>
@@
 <part name="FRAME1" library="SparkFun-Aesthetics" library_urn="urn:adsk.eagle:library:507" deviceset="FRAME-A4L" device=""/>
 <part name="P+1" library="supply1" library_urn="urn:adsk.eagle:library:371" deviceset="+12V" device=""/>
+<part name="S1" library="SparkFun-Switches" deviceset="MOMENTARY-SWITCH-SPST" device="-PTH-6.0MM"/>
+<part name="SUPPLY3" library="supply2" deviceset="GND" device=""/>
 </parts>
 <sheets>
@@
 <instance part="P+1" gate="1" x="109.22" y="124.46" smashed="yes">
 <attribute name="VALUE" x="106.68" y="119.38" size="1.778" layer="96" rot="R90"/>
+</instance>
+<instance part="S1" gate="G$1" x="27.94" y="38.1" smashed="yes" rot="R90">
+<attribute name="NAME" x="26.416" y="38.1" size="1.778" layer="95" font="vector" rot="R90" align="bottom-center"/>
+<attribute name="VALUE" x="30.988" y="38.1" size="1.778" layer="96" font="vector" rot="R270" align="top-center"/>
+</instance>
+<instance part="SUPPLY3" gate="GND" x="27.94" y="10.16" smashed="yes">
+<attribute name="VALUE" x="26.035" y="6.985" size="1.778" layer="96"/>
 </instance>
 </instances>
@@
 <junction x="137.16" y="55.88"/>
 </segment>
+<segment>
+<pinref part="S1" gate="G$1" pin="1"/>
+<pinref part="SUPPLY3" gate="GND" pin="GND"/>
+<wire x1="27.94" y1="33.02" x2="27.94" y2="12.7" width="0.1524" layer="91"/>
+</segment>
 </net>
 <net name="VCC" class="2">
@@
 </segment>
 </net>
+<net name="N$1" class="0">
+<segment>
+<pinref part="MC1" gate="G$1" pin="2"/>
+<pinref part="S1" gate="G$1" pin="2"/>
+<wire x1="27.94" y1="53.34" x2="27.94" y2="43.18" width="0.1524" layer="91"/>
+</segment>
+</net>
